File: PCB/mouse_v1/mouse_v1.kicad_sch (KiCad schematic)
At the start: 27 parts, among them IC1 NJM7805FA, IC2 SIT2001BI-S2-33E-12.000000G, J1 Conn_01x06_Socket, J2 Conn_01x06_Socket, Q1 2SC1815GRTE2FT, Q2 2SJ681_Q_, Q3 2SJ681_Q_, U1 NUCLEO-L432KC, U2 SLA7073MPRT, U3 SLA7073MPRT

Commit message: 回路図のデータ作成終了,名前振り開始
Parts:
- added C11, C12: C_Polarized_Small, symbol Device:C_Polarized_Small
- added D2: D, symbol Device:D
- added D3: LED, symbol Device:LED
- added J3: Conn_01x02_Socket, symbol Connector:Conn_01x02_Socket
- added LED1, LED2, LED3, LED4: OS5RKA5111P, OS5RKA5111P, symbol OS5RKA5111P:OS5RKA5111P
- added LS1: QMB-111GPN, QMB111GPN, symbol QMB-111GPN:QMB-111GPN
- added Q4, Q5, Q6, Q7: ST-1KL3A, ST1KL3A, symbol ST-1KL3A:ST-1KL3A
- added Q8, Q9: 2SC1815GRTE2FT, 2SC1815GRTE2FT, symbol 2SC1815GRTE2FT:2SC1815GRTE2FT
- added R10, R11, R12, R13, R14, R15, R16, R17, R18, R19, R5, R6, R7, R8, R9: R, symbol Device:R
- added SW1, SW2: SW_Push, symbol Switch:SW_Push
- added SW4: SW_DIP_x01, symbol Switch:SW_DIP_x01
Connections:
- net +12V: now also C1.1, C2.1, IC1.1 (IN), Q2.2 (DRAIN), R18.1
- net +3.3V: now also D2.1 (K), LS1.2, Q4.2 (C), Q5.2 (C), Q6.2 (C), Q7.2 (C)
- net +5V: now also C3.1, C4.1, IC1.3 (OUT), R14.1, R9.1
- net BATTERY: now also R18.2, R19.1
- net GND: now also C1.2, C2.2, C3.2, C4.2, IC1.2 (GND), Q1.1 (E), C11.2, C12.2, J3.2 (Pin_2), Q8.1 (E), Q9.1 (E), R10.2, R13.2, R16.1, R17.2, R19.2, R5.2, R6.2, R7.2, R8.2, SW1.1, SW2.1, SW4.1
- net INTERFACELED: now also D3.2 (A)
- net SENSORLED_1: now also R11.2, R12.2
- net SPEAKER: now also R15.2
- net SWITCH_1: now also SW1.2
- net SWITCH_2: now also SW2.2
- net photosensor_2: now also Q5.1 (E), R6.1
- net photosensor_3: now also Q6.1 (E), R7.1
- net photosensor_4: now also Q7.1 (E), R8.1
- net at Q1.2 (C): now also LED1.1 (K)
- net at Q1.3 (B): now also R10.1, R11.1
- net at R1.1: now also D1.2 (A), Q2.1 (GATE)
- net at R1.2: now also Q2.3 (SOURCE), J3.1 (Pin_1)
- net at D1.1 (K): now also SW4.2
- net photosensor1 renamed photosensor_1
- net photosensor_1: now also Q4.1 (E), R5.1
- new net: Q8.3 (B), R12.1, R13.1
- new net: C12.1, LED3.2 (A), R14.2
- new net: Q9.3 (B), R15.1, R16.2
- new net: LED3.1 (K), LED4.2 (A)
- new net: LED1.2 (A), LED2.1 (K)
- new net: C11.1, LED2.2 (A), R9.2
- new net: D3.1 (K), R17.1
- new net: D2.2 (A), LS1., Q9.2 (C)
- new net: LED4.1 (K), Q8.2 (C)
Other:
- note added: "Clock"
- moved on the sheet: C1, C2, C3, C4, D1, IC1, Q1, R1

Commit message: 回路図の名前振り終了
Other:
- note added: "Buzzer"
- note added: "Check"
- note added: "Main"
- note added: "Motor_Driver"
- note added: "Power"
- note added: "connect"
- note added: "photo-sensor"
- moved on the sheet: C1, C10, C11, C12, C2, C3, C4, C6, C7, C8, C9, D1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

Commit message: capactorを適当にフットプリント振った
Parts:
- C1, C10, C11, C12, C2, C3, C4, C5, C6, C7, C8, C9: footprint (none) -> Capacitor_SMD:C_0603_1608Metric
- D1, D3: footprint (none) -> LED_SMD:LED_0603_1608Metric
- D2: footprint (none) -> Diode_SMD:D_0603_1608Metric
Changed lines of the file:
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@@
       (effects (font (size 1.27 1.27)) (justify left))
     )
-    (property "Footprint" "" (at 72.0852 274.32 0)
+    (property "Footprint" "Capacitor_SMD:C_0603_1608Metric" (at 72.0852 274.32 0)
       (effects (font (size 1.27 1.27)) hide)
     )
@@
       (effects (font (size 1.27 1.27)) (justify left))
     )
-    (property "Footprint" "" (at 119.38 78.74 0)
+    (property "Footprint" "Capacitor_SMD:C_0603_1608Metric" (at 119.38 78.74 0)
       (effects (font (size 1.27 1.27)) hide)
     )
@@
       (effects (font (size 1.27 1.27)) (justify left))
     )
-    (property "Footprint" "" (at 328.93 46.99 0)
+    (property "Footprint" "Capacitor_SMD:C_0603_1608Metric" (at 328.93 46.99 0)
       (effects (font (size 1.27 1.27)) hide)
     )
@@
       (effects (font (size 1.27 1.27)))
     )
-    (property "Footprint" "" (at 35.56 74.93 0)
+    (property "Footprint" "LED_SMD:LED_0603_1608Metric" (at 35.56 74.93 0)
       (effects (font (size 1.27 1.27)) hide)
     )
@@
       (effects (font (size 1.27 1.27)) (justify left))
     )
-    (property "Footprint" "" (at 346.71 237.49 0)
+    (property "Footprint" "Capacitor_SMD:C_0603_1608Metric" (at 346.71 237.49 0)
       (effects (font (size 1.27 1.27)) hide)
     )
@@
       (effects (font (size 1.27 1.27)) (justify right))
     )
-    (property "Footprint" "" (at 66.04 220.98 0)
+    (property "Footprint" "LED_SMD:LED_0603_1608Metric" (at 66.04 220.98 0)
       (effects (font (size 1.27 1.27)) hide)
     )
@@
       (effects (font (size 1.27 1.27)) (justify left))
     )
-    (property "Footprint" "" (at 222.25 140.97 0)
+    (property "Footprint" "Diode_SMD:D_0603_1608Metric" (at 222.25 140.97 0)
       (effects (font (size 1.27 1.27)) hide)
     )
@@
       (effects (font (size 1.27 1.27)) (justify left))
     )
-    (property "Footprint" "" (at 110.1852 82.55 0)
+    (property "Footprint" "Capacitor_SMD:C_0603_1608Metric" (at 110.1852 82.55 0)
       (effects (font (size 1.27 1.27)) hide)
     )
@@
       (effects (font (size 1.27 1.27)) (justify left))
     )
-    (property "Footprint" "" (at 382.27 66.04 0)
+    (property "Footprint" "Capacitor_SMD:C_0603_1608Metric" (at 382.27 66.04 0)
       (effects (font (size 1.27 1.27)) hide)
     )
@@
       (effects (font (size 1.27 1.27)) (justify left))
     )
-    (property "Footprint" "" (at 304.4952 201.93 0)
+    (property "Footprint" "Capacitor_SMD:C_0603_1608Metric" (at 304.4952 201.93 0)
       (effects (font (size 1.27 1.27)) hide)
     )
@@
       (effects (font (size 1.27 1.27)) (justify left))
     )
-    (property "Footprint" "" (at 368.3 237.49 0)
+    (property "Footprint" "Capacitor_SMD:C_0603_1608Metric" (at 368.3 237.49 0)
       (effects (font (size 1.27 1.27)) hide)
     )
@@
       (effects (font (size 1.27 1.27)) (justify left))
     )
-    (property "Footprint" "" (at 92.4052 82.55 0)
+    (property "Footprint" "Capacitor_SMD:C_0603_1608Metric" (at 92.4052 82.55 0)
       (effects (font (size 1.27 1.27)) hide)
     )
@@
       (effects (font (size 1.27 1.27)) (justify right))
     )
-    (property "Footprint" "" (at 352.0948 160.02 0)
+    (property "Footprint" "Capacitor_SMD:C_0603_1608Metric" (at 352.0948 160.02 0)
       (effects (font (size 1.27 1.27)) hide)
     )
@@
       (effects (font (size 1.27 1.27)) (justify left))
     )
-    (property "Footprint" "" (at 80.01 74.93 0)
+    (property "Footprint" "Capacitor_SMD:C_0603_1608Metric" (at 80.01 74.93 0)
       (effects (font (size 1.27 1.27)) hide)
     )
@@
       (effects (font (size 1.27 1.27)))
     )
-    (property "Footprint" "" (at 354.33 153.9748 0)
-      (effects (font (size 1.27 1.27)) hide)
-    )
+    (property "Footprint" "Capacitor_SMD:C_0603_1608Metric" (at 354.33 153.9748 0)
+      (effects (font (size 1.27 1.27)) hide)
+    )

Commit message: フットプリントを途中まで割り当てて,外部からインポートした部品はできていない
Parts:
- DS1: footprint AQM0802ARNGBW -> (none)
- IC1: footprint TO254P500X1000X2170-3P -> (none)
- IC2: footprint SOT95P280X130-5N -> (none)
- J1, J2: footprint (none) -> Connector_JST:JST_XH_B6B-XH-A_1x06_P2.50mm_Vertical
- J3: footprint (none) -> Connector_JST:JST_XH_B2B-XH-A_1x02_P2.50mm_Vertical
- LED1, LED2, LED3, LED4: footprint OS5RKA5111P -> LED_THT:LED_D5.0mm
- LS1: footprint QMB111GPN -> (none)
- Q1, Q8, Q9: footprint 2SC1815GRTE2FT -> (none)
- Q2, Q3: footprint TO230P250X650X900-3P -> (none)
- Q4, Q5, Q6, Q7: footprint ST1KL3A -> (none)
- R1, R10, R11, R12, R13, R14, R15, R16, R17, R18, R19, R2, R3, R4, R5, R6, R7, R8, R9: footprint (none) -> Resistor_SMD:R_0603_1608Metric_Pad0.98x0.95mm_HandSolder
- SW1, SW2: footprint (none) -> Button_Switch_THT:SW_PUSH_6mm_H7.3mm
- SW4: footprint (none) -> Button_Switch_THT:SW_DIP_SPSTx01_Slide_9.78x4.72mm_W7.62mm_P2.54mm
- VR1: footprint 3296W1102LF -> (none)

Commit message: 基板のフットプリント完了
Parts:
- DS1: footprint (none) -> AQM0802A-RN-GBW:AQM0802ARNGBW
- IC1: footprint (none) -> NJM7805FA:TO254P500X1000X2170-3P
- IC2: footprint (none) -> SIT2001BI-S2-33E-12.000000G:SOT95P280X130-5N
- LED1, LED2, LED3, LED4: footprint LED_THT:LED_D5.0mm -> OS5RKA5111P:OS5RKA5111P
- LS1: footprint (none) -> QMB111GPN
- Q1, Q8, Q9: footprint (none) -> 2SC1815GRTE2FT:2SC1815GRTE2FT
- Q2, Q3: footprint (none) -> 2SJ681_Q_:TO230P250X650X900-3P
- Q4, Q5, Q6, Q7: footprint (none) -> ST-1KL3A:ST1KL3A
- U2, U3: footprint (none) -> SLA7073MPRT:SLA7073MPRT
- VR1: footprint (none) -> 3296W-1-102LF:3296W1102LF
Connections:
- net at D2.2 (A), Q9.2 (C): now also LS1.1; no longer LS1.
Changed lines of the file:
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@@
       (effects (font (size 1.27 1.27)) (justify left))
     )
-    (property "Footprint" "" (at 220.98 243.84 0)
+    (property "Footprint" "SLA7073MPRT:SLA7073MPRT" (at 220.98 243.84 0)
       (effects (font (size 1.27 1.27) italic) hide)
     )
@@
       (effects (font (size 1.27 1.27)) (justify left))
     )
-    (property "Footprint" "" (at 161.29 162.23 0)
+    (property "Footprint" "ST-1KL3A:ST1KL3A" (at 161.29 162.23 0)
       (effects (font (size 1.27 1.27)) (justify left top) hide)
     )
@@
       (effects (font (size 1.27 1.27)) (justify left))
     )
-    (property "Footprint" "" (at 213.36 160.96 0)
+    (property "Footprint" "ST-1KL3A:ST1KL3A" (at 213.36 160.96 0)
       (effects (font (size 1.27 1.27)) (justify left top) hide)
     )
@@
       (effects (font (size 1.27 1.27)) (justify right))
     )
-    (property "Footprint" "" (at 388.29 152.4 0)
+    (property "Footprint" "2SJ681_Q_:TO230P250X650X900-3P" (at 388.29 152.4 0)
       (effects (font (size 1.27 1.27)) (justify left top) hide)
     )
@@
       (effects (font (size 1.27 1.27)) (justify left))
     )
-    (property "Footprint" "" (at 363.22 218.11 0)
+    (property "Footprint" "2SC1815GRTE2FT:2SC1815GRTE2FT" (at 363.22 218.11 0)
       (effects (font (size 1.27 1.27)) (justify left top) hide)
     )
@@
       (effects (font (size 1.27 1.27)) (justify right))
     )
-    (property "Footprint" "LED_THT:LED_D5.0mm" (at 399.72 50.8 0)
+    (property "Footprint" "OS5RKA5111P:OS5RKA5111P" (at 399.72 50.8 0)
       (effects (font (size 1.27 1.27)) (justify left bottom) hide)
     )
@@
       (effects (font (size 1.27 1.27)) (justify left))
     )
-    (property "Footprint" "" (at 152.4 243.84 0)
+    (property "Footprint" "SLA7073MPRT:SLA7073MPRT" (at 152.4 243.84 0)
       (effects (font (size 1.27 1.27) italic) hide)
     )
@@
       (effects (font (size 1.27 1.27)) (justify right))
     )
-    (property "Footprint" "LED_THT:LED_D5.0mm" (at 453.06 69.85 0)
+    (property "Footprint" "OS5RKA5111P:OS5RKA5111P" (at 453.06 69.85 0)
       (effects (font (size 1.27 1.27)) (justify left bottom) hide)
     )
@@
     )
   )
+  (symbol (lib_id "QMB-111GPN:QMB-111GPN") (at 196.85 144.78 0) (mirror y) (unit 1)
+    (in_bom yes) (on_board yes) (dnp no) (fields_autoplaced)
+    (property "Reference" "LS1" (at 189.484 135.89 0)
+      (effects (font (size 1.27 1.27)))
+    )
+    (property "Value" "QMB-111GPN" (at 189.484 138.43 0)
+      (effects (font (size 1.27 1.27)))
+    )
+    (property "Footprint" "QMB111GPN" (at 185.42 247.32 0)
+      (effects (font (size 1.27 1.27)) (justify left top) hide)
+    )
+    (property "Datasheet" "" (at 185.42 347.32 0)
+      (effects (font (size 1.27 1.27)) (justify left top) hide)
+    )
+    (property "Height" "8.5" (at 185.42 547.32 0)
+      (effects (font (size 1.27 1.27)) (justify left top) hide)
+    )
+    (property "RS Part Number" "" (at 185.42 647.32 0)
+      (effects (font (size 1.27 1.27)) (justify left top) hide)
+    )
+    (property "RS Price/Stock" "" (at 185.42 747.32 0)
+      (effects (font (size 1.27 1.27)) (justify left top) hide)
+    )
+    (property "Manufacturer_Name" "Star Micronics LTD" (at 185.42 847.32 0)
+      (effects (font (size 1.27 1.27)) (justify left top) hide)
+    )
+    (property "Manufacturer_Part_Number" "QMB-111GPN" (at 185.42 947.32 0)
+      (effects (font (size 1.27 1.27)) (justify left top) hide)
+    )
+    (pin "1")
+    (pin "2")
+    (instances
+      (project "mouse_v1"
+        (path "/6382fc59-4609-4144-a48b-8e85eb517642"
+          (reference "LS1") (unit 1)
+        )
+      )
+    )
+  )
   (symbol (lib_id "power:GND") (at 44.45 205.74 0) (unit 1)
     (in_bom yes) (on_board yes) (dnp no) (fields_autoplaced)
@@
       (effects (font (size 1.27 1.27)) (justify left))
     )
-    (property "Footprint" "" (at 240.03 160.96 0)
+    (property "Footprint" "ST-1KL3A:ST1KL3A" (at 240.03 160.96 0)
       (effects (font (size 1.27 1.27)) (justify left top) hide)
     )
@@
       (effects (font (size 1.27 1.27)) (justify right))
     )
-    (property "Footprint" "" (at 139.37 35.56 0)
+    (property "Footprint" "2SJ681_Q_:TO230P250X650X900-3P" (at 139.37 35.56 0)
       (effects (font (size 1.27 1.27)) (justify left top) hide)
     )
@@
       (effects (font (size 1.27 1.27)) (justify left))
     )
-    (property "Footprint" "" (at 389.89 253.67 0)
+    (property "Footprint" "AQM0802A-RN-GBW:AQM0802ARNGBW" (at 389.89 253.67 0)
       (effects (font (size 1.27 1.27)) (justify left top) hide)
     )
@@
       (effects (font (size 1.27 1.27)))
     )
-    (property "Footprint" "" (at 60.96 355.27 0)
+    (property "Footprint" "SIT2001BI-S2-33E-12.000000G:SOT95P280X130-5N" (at 60.96 355.27 0)
       (effects (font (size 1.27 1.27)) (justify left top) hide)
     )
@@
       (effects (font (size 1.27 1.27)) (justify left))
     )
-    (property "Footprint" "" (at 186.69 160.96 0)
+    (property "Footprint" "ST-1KL3A:ST1KL3A" (at 186.69 160.96 0)
       (effects (font (size 1.27 1.27)) (justify left top) hide)
     )
@@
       (effects (font (size 1.27 1.27)) (justify left))
     )
-    (property "Footprint" "" (at 335.28 286.69 0)
+    (property "Footprint" "3296W-1-102LF:3296W1102LF" (at 335.28 286.69 0)
       (effects (font (size 1.27 1.27)) (justify left top) hide)
     )
@@
       (effects (font (size 1.27 1.27)) (justify right))
     )
-    (property "Footprint" "LED_THT:LED_D5.0mm" (at 453.06 91.44 0)
+    (property "Footprint" "OS5RKA5111P:OS5RKA5111P" (at 453.06 91.44 0)
       (effects (font (size 1.27 1.27)) (justify left bottom) hide)
     )
@@
     )
   )
-  (symbol (lib_id "QMB-111GPN:QMB-111GPN") (at 196.85 144.78 0) (mirror y) (unit 1)
-    (in_bom yes) (on_board yes) (dnp no)
-    (property "Reference" "LS1" (at 185.42 144.78 0)
-      (effects (font (size 1.27 1.27)) (justify left))
-    )
-    (property "Value" "QMB-111GPN" (at 185.42 147.32 0)
-      (effects (font (size 1.27 1.27)) (justify left))
-    )
-    (property "Footprint" "" (at 185.42 247.32 0)
-      (effects (font (size 1.27 1.27)) (justify left top) hide)
-    )
-    (property "Datasheet" "" (at 185.42 347.32 0)
-      (effects (font (size 1.27 1.27)) (justify left top) hide)
-    )
-    (property "Height" "8.5" (at 185.42 547.32 0)
-      (effects (font (size 1.27 1.27)) (justify left top) hide)
-    )
-    (property "RS Part Number" "" (at 185.42 647.32 0)
-      (effects (font (size 1.27 1.27)) (justify left top) hide)
-    )
-    (property "RS Price/Stock" "" (at 185.42 747.32 0)
-      (effects (font (size 1.27 1.27)) (justify left top) hide)
-    )
-    (property "Manufacturer_Name" "Star Micronics LTD" (at 185.42 847.32 0)
-      (effects (font (size 1.27 1.27)) (justify left top) hide)
-    )
-    (property "Manufacturer_Part_Number" "QMB-111GPN" (at 185.42 947.32 0)
-      (effects (font (size 1.27 1.27)) (justify left top) hide)
-    )
-    (pin "2")
-    (pin "")
-    (instances
-      (project "mouse_v1"
-        (path "/6382fc59-4609-4144-a48b-8e85eb517642"
-          (reference "LS1") (unit 1)
-        )
-      )
-    )
-  )
   (symbol (lib_id "Switch:SW_Push") (at 53.34 205.74 0) (unit 1)
     (in_bom yes) (on_board yes) (dnp no) (fields_autoplaced)
@@
       (effects (font (size 1.27 1.27)) (justify left))
     )
-    (property "Footprint" "" (at 212.09 262.56 0)
+    (property "Footprint" "2SC1815GRTE2FT:2SC1815GRTE2FT" (at 212.09 262.56 0)
       (effects (font (size 1.27 1.27)) (justify left top) hide)
     )
@@
       (effects (font (size 1.27 1.27)) (justify left))
     )
-    (property "Footprint" "" (at 309.88 199.06 0)
+    (property "Footprint" "2SC1815GRTE2FT:2SC1815GRTE2FT" (at 309.88 199.06 0)
       (effects (font (size 1.27 1.27)) (justify left top) hide)
     )
@@
       (effects (font (size 1.27 1.27)) (justify right))
     )
-    (property "Footprint" "LED_THT:LED_D5.0mm" (at 399.72 72.39 0)
+    (property "Footprint" "OS5RKA5111P:OS5RKA5111P" (at 399.72 72.39 0)
       (effects (font (size 1.27 1.27)) (justify left bottom) hide)
     )
@@
       (effects (font (size 1.27 1.27)) (justify right))
     )
-    (property "Footprint" "" (at 192.71 44.45 0)
-      (effects (font (size 1.27 1.27)) (justify left top) hide)
-    )
+    (property "Footprint" "NJM7805FA:TO254P500X1000X2170-3P" (at 192.71 44.45 0)
+      (effects (font (size 1.27 1.27)) (justify left top) hide)
+    )
