File: PCB/mouse_v1/mouse_v1.kicad_sch (KiCad schematic)
At the start: 61 parts, among them IC1 NJM7805FA, IC2 SIT2001BI-S2-33E-12.000000G, J1 Conn_01x06_Socket, J2 Conn_01x06_Socket, J3 Conn_01x02_Socket, Q1 2SC1815GRTE2FT, Q2 2SJ681_Q_, Q3 2SJ681_Q_, Q4 ST-1KL3A, Q5 ST-1KL3A, Q6 ST-1KL3A, Q7 ST-1KL3A, Q8 2SC1815GRTE2FT, Q9 2SC1815GRTE2FT, SW1 SW_Push, SW2 SW_Push, SW4 SW_DIP_x01, U1 NUCLEO-L432KC, U2 SLA7073MPRT, U3 SLA7073MPRT

Commit message: 抵抗やコンデンサに具体的な値を明示した
Parts:
- C1, C10, C3, C6, C9: value C -> 0.1μ
- C11, C12, C2, C4, C7, C8: value C_Polarized_Small -> 100μ
- C5: value C -> 15p
- D2: value D -> BA157
- R1, R10, R13, R16, R2, R3, R4: value R -> 10K
- R11, R12, R15, R5, R6, R7, R8: value R -> 4.7K
- R14, R9: value R -> 50K
- R18: value R -> 100K
- R19: value R -> 22K
- renumbered R17 to 1K
Other:
- note added: "LED"
Changed lines of the file:
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@@
     (effects (font (size 5 5) bold) (justify left bottom))
   )
-  (text "Buzzer" (at 267.97 27.94 0)
+  (text "LED" (at 267.97 27.94 0)
     (effects (font (size 5 5) bold) (justify left bottom))
   )
@@
       (effects (font (size 1.27 1.27)) (justify left))
     )
-    (property "Value" "C" (at 74.93 271.78 0)
+    (property "Value" "15p" (at 74.93 271.78 0)
       (effects (font (size 1.27 1.27)) (justify left))
     )
@@
       (effects (font (size 1.27 1.27)) (justify left))
     )
-    (property "Value" "R" (at 293.37 106.68 0)
+    (property "Value" "10K" (at 293.37 106.68 0)
       (effects (font (size 1.27 1.27)) (justify left))
     )
@@
       (effects (font (size 1.27 1.27)))
     )
-    (property "Value" "R" (at 284.48 93.98 90)
+    (property "Value" "4.7K" (at 284.48 93.98 90)
       (effects (font (size 1.27 1.27)))
     )
@@
       (effects (font (size 1.27 1.27)) (justify left))
     )
-    (property "Value" "C_Polarized_Small" (at 121.92 79.4639 0)
+    (property "Value" "100μ" (at 121.92 79.4639 0)
       (effects (font (size 1.27 1.27)) (justify left))
     )
@@
       (effects (font (size 1.27 1.27)) (justify left))
     )
-    (property "Value" "R" (at 73.66 86.36 0)
+    (property "Value" "22K" (at 73.66 86.36 0)
       (effects (font (size 1.27 1.27)) (justify left))
     )
@@
       (effects (font (size 1.27 1.27)) (justify left))
     )
-    (property "Value" "R" (at 160.02 87.63 0)
+    (property "Value" "4.7K" (at 160.02 87.63 0)
       (effects (font (size 1.27 1.27)) (justify left))
     )
@@
       (effects (font (size 1.27 1.27)) (justify left))
     )
-    (property "Value" "R" (at 346.71 125.73 0)
+    (property "Value" "10K" (at 346.71 125.73 0)
       (effects (font (size 1.27 1.27)) (justify left))
     )
@@
       (effects (font (size 1.27 1.27)) (justify left))
     )
-    (property "Value" "R" (at 308.61 39.37 0)
+    (property "Value" "50K" (at 308.61 39.37 0)
       (effects (font (size 1.27 1.27)) (justify left))
     )
@@
       (effects (font (size 1.27 1.27)) (justify right))
     )
-    (property "Value" "R" (at 195.58 171.45 0)
+    (property "Value" "10K" (at 195.58 171.45 0)
       (effects (font (size 1.27 1.27)) (justify right))
     )
@@
       (effects (font (size 1.27 1.27)) (justify left))
     )
-    (property "Value" "C_Polarized_Small" (at 331.47 47.7139 0)
+    (property "Value" "100μ" (at 331.47 47.7139 0)
       (effects (font (size 1.27 1.27)) (justify left))
     )
@@
       (effects (font (size 1.27 1.27)) (justify left))
     )
-    (property "Value" "R" (at 295.91 186.69 0)
+    (property "Value" "10K" (at 295.91 186.69 0)
       (effects (font (size 1.27 1.27)) (justify left))
     )
@@
       (effects (font (size 1.27 1.27)) (justify left))
     )
-    (property "Value" "R" (at 73.66 73.66 0)
+    (property "Value" "100K" (at 73.66 73.66 0)
       (effects (font (size 1.27 1.27)) (justify left))
     )
@@
       (effects (font (size 1.27 1.27)) (justify left))
     )
-    (property "Value" "R" (at 25.4 66.04 0)
+    (property "Value" "10K" (at 25.4 66.04 0)
       (effects (font (size 1.27 1.27)) (justify left))
     )
@@
       (effects (font (size 1.27 1.27)) (justify left))
     )
-    (property "Value" "R" (at 238.76 86.36 0)
+    (property "Value" "4.7K" (at 238.76 86.36 0)
       (effects (font (size 1.27 1.27)) (justify left))
     )
@@
       (effects (font (size 1.27 1.27)) (justify left))
     )
-    (property "Value" "R" (at 309.88 180.34 0)
+    (property "Value" "10K" (at 309.88 180.34 0)
       (effects (font (size 1.27 1.27)) (justify left))
     )
@@
       (effects (font (size 1.27 1.27)) (justify left))
     )
-    (property "Value" "R" (at 185.42 86.36 0)
+    (property "Value" "4.7K" (at 185.42 86.36 0)
       (effects (font (size 1.27 1.27)) (justify left))
     )
@@
       (effects (font (size 1.27 1.27)) (justify left))
     )
-    (property "Value" "C_Polarized_Small" (at 349.25 238.2139 0)
+    (property "Value" "100μ" (at 349.25 238.2139 0)
       (effects (font (size 1.27 1.27)) (justify left))
     )
@@
       (effects (font (size 1.27 1.27)) (justify left))
     )
-    (property "Value" "D" (at 224.79 142.24 90)
+    (property "Value" "BA157" (at 224.79 142.24 90)
       (effects (font (size 1.27 1.27)) (justify left))
     )
@@
       (effects (font (size 1.27 1.27)))
     )
-    (property "Value" "R" (at 184.15 157.48 90)
+    (property "Value" "4.7K" (at 184.15 157.48 90)
       (effects (font (size 1.27 1.27)))
     )
@@
       (effects (font (size 1.27 1.27)) (justify left))
     )
-    (property "Value" "C" (at 113.03 80.01 0)
+    (property "Value" "0.1μ" (at 113.03 80.01 0)
       (effects (font (size 1.27 1.27)) (justify left))
     )
@@
       (effects (font (size 1.27 1.27)) (justify left))
     )
-    (property "Value" "R" (at 361.95 58.42 0)
+    (property "Value" "50K" (at 361.95 58.42 0)
       (effects (font (size 1.27 1.27)) (justify left))
     )
@@
       (effects (font (size 1.27 1.27)))
     )
-    (property "Value" "R" (at 349.25 176.53 90)
+    (property "Value" "10K" (at 349.25 176.53 90)
       (effects (font (size 1.27 1.27)))
     )
@@
       (effects (font (size 1.27 1.27)) (justify left))
     )
-    (property "Value" "C_Polarized_Small" (at 384.81 66.7639 0)
+    (property "Value" "100μ" (at 384.81 66.7639 0)
       (effects (font (size 1.27 1.27)) (justify left))
     )
@@
       (effects (font (size 1.27 1.27)) (justify left))
     )
-    (property "Value" "C" (at 307.34 199.39 0)
+    (property "Value" "0.1μ" (at 307.34 199.39 0)
       (effects (font (size 1.27 1.27)) (justify left))
     )
@@
   (symbol (lib_id "Device:R") (at 54.61 220.98 270) (mirror x) (unit 1)
     (in_bom yes) (on_board yes) (dnp no) (fields_autoplaced)
-    (property "Reference" "R17" (at 55.88 218.44 0)
-      (effects (font (size 1.27 1.27)) (justify left))
+    (property "Reference" "1K" (at 54.61 214.63 90)
+      (effects (font (size 1.27 1.27)))
     )
-    (property "Value" "R" (at 53.34 218.44 0)
-      (effects (font (size 1.27 1.27)) (justify left))
+    (property "Value" "R" (at 54.61 217.17 90)
+      (effects (font (size 1.27 1.27)))
     )
     (property "Footprint" "Resistor_SMD:R_0603_1608Metric_Pad0.98x0.95mm_HandSolder" (at 54.61 222.758 90)
@@
       (project "mouse_v1"
         (path "/6382fc59-4609-4144-a48b-8e85eb517642"
-          (reference "R17") (unit 1)
+          (reference "1K") (unit 1)
         )
       )
@@
       (effects (font (size 1.27 1.27)) (justify left))
     )
-    (property "Value" "C_Polarized_Small" (at 370.84 238.2139 0)
+    (property "Value" "100μ" (at 370.84 238.2139 0)
       (effects (font (size 1.27 1.27)) (justify left))
     )
@@
       (effects (font (size 1.27 1.27)))
     )
-    (property "Value" "R" (at 337.82 113.03 90)
+    (property "Value" "4.7K" (at 337.82 113.03 90)
       (effects (font (size 1.27 1.27)))
     )
@@
       (effects (font (size 1.27 1.27)) (justify left))
     )
-    (property "Value" "R" (at 212.09 86.36 0)
+    (property "Value" "4.7K" (at 212.09 86.36 0)
       (effects (font (size 1.27 1.27)) (justify left))
     )
@@
       (effects (font (size 1.27 1.27)) (justify left))
     )
-    (property "Value" "C" (at 95.25 80.01 0)
+    (property "Value" "0.1μ" (at 95.25 80.01 0)
       (effects (font (size 1.27 1.27)) (justify left))
     )
@@
       (effects (font (size 1.27 1.27)) (justify right))
     )
-    (property "Value" "C" (at 356.87 165.1 0)
+    (property "Value" "0.1μ" (at 356.87 165.1 0)
       (effects (font (size 1.27 1.27)) (justify right))
     )
@@
       (effects (font (size 1.27 1.27)) (justify left))
     )
-    (property "Value" "C_Polarized_Small" (at 82.55 75.6539 0)
+    (property "Value" "100μ" (at 82.55 75.6539 0)
       (effects (font (size 1.27 1.27)) (justify left))
     )
@@
       (effects (font (size 1.27 1.27)))
     )
-    (property "Value" "C" (at 350.52 149.86 90)
+    (property "Value" "0.1μ" (at 350.52 149.86 90)
       (effects (font (size 1.27 1.27)))
     )
