File: PCB/mouse_v1/mouse_v1.kicad_sch (KiCad schematic)
At the start: 61 parts, among them IC1 NJM7805FA, IC2 SIT2001BI-S2-33E-12.000000G, J1 Conn_01x06_Socket, J2 Conn_01x06_Socket, J3 Conn_01x02_Socket, Q1 2SC1815GRTE2FT, Q2 2SJ681_Q_, Q3 2SJ681_Q_, Q4 ST-1KL3A, Q5 ST-1KL3A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

Commit message: 配線完了(仮)
Parts:
- C11, C12, C2, C4, C7, C8: footprint Capacitor_SMD:C_0603_1608Metric -> Capacitor_THT:CP_Radial_D6.3mm_P2.50mm
- Q1, Q8, Q9: footprint 2SC1815GRTE2FT:2SC1815GRTE2FT -> Package_TO_SOT_SMD:SOT-23
Connections:
- net SENSORLED_1: no longer R11.2
- net SENSORLED_2: now also R11.2
