File: PCB/mouse_v1/_autosave-mouse_v1.kicad_sch (KiCad schematic)
At the start: 61 parts, among them IC1 NJM7805FA, IC2 SIT2001BI-S2-33E-12.000000G, J1 Conn_01x06_Socket, J2 Conn_01x06_Socket, J3 Conn_01x02_Socket, Q1 2SC1815GRTE2FT, Q2 2SJ681_Q_, Q3 2SJ681_Q_, Q4 ST-1KL3A, Q5 ST-1KL3A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

Commit message: 配線完了,元のデータはsensorLEDのフラグの値が両方1になっていた
Connections:
- net SENSORLED_1: no longer R11.2
- net SENSORLED_2: now also R11.2
Changed lines of the file:
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@@
     )
   )
-  (global_label "SENSORLED_1" (shape input) (at 334.01 116.84 180) (fields_autoplaced)
+  (global_label "SENSORLED_2" (shape input) (at 334.01 116.84 180) (fields_autoplaced)
     (effects (font (size 1.27 1.27)) (justify right))
     (property "Intersheetrefs" "${INTERSHEET_REFS}" (at 317.9016 116.84 0)
