File: PCB/mouse_v1/mouse_v1.kicad_pcb (KiCad board)
At the start: 2 copper layers, 61 parts, among them IC1 NJM7805FA, IC2 SIT2001BI-S2-33E-12.000000G, J1 Conn_01x06_Socket, J2 Conn_01x06_Socket, J3 Conn_01x02_Socket, Q1 2SC1815GRTE2FT, Q2 2SJ681_Q_, Q3 2SJ681_Q_, Q4 ST-1KL3A, Q5 ST-1KL3A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

Commit message: 配線が短くなるように配線した,I2Cは長くなった
Parts:
- J1, J2, LED1, LED2, LED3, LED4, Q4, Q5, Q6, Q7: moved to B.Cu
- moved R9 273.3 mm to (91.4, 86.4), turned to 90 degrees
- moved C11 270.2 mm to (94.0, 86.4), turned to -90 degrees
- moved R11 237.6 mm to (128.6, 91.4), turned to 180 degrees
- moved LED2 236.3 mm to (114.3, 66.0), turned to 120 degrees
- moved R10 233.5 mm to (133.7, 91.4)
- moved Q1 229.5 mm to (139.7, 83.8)
- moved LED1 221.9 mm to (134.6, 76.6), turned to 170 degrees
- moved C8 191.4 mm to (86.4, 147.3), turned to -90 degrees
- moved J2 186.6 mm to (81.3, 147.3), turned to 180 degrees
- moved C7 186.3 mm to (91.4, 147.3), turned to -90 degrees
- moved C10 180.9 mm to (108.4, 84.7), turned to 180 degrees
- moved C9 176.7 mm to (111.8, 86.4), turned to 180 degrees
- moved R12 171.7 mm to (78.7, 86.4)
- moved DS1 171.6 mm to (104.8, 79.7)
- moved R14 170.2 mm to (88.9, 86.4), turned to 90 degrees
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
Commit message: 配線完了した(埋め込んだcadがおかしいかも)
Parts:
- moved D2 20.9 mm to (119.4, 112.5)
- moved LS1 20.5 mm to (109.2, 119.4), turned to 0 degrees
- moved SW1 20.3 mm to (99.8, 116.5)
- moved SW2 20.3 mm to (89.6, 116.3)
- moved R15 18.0 mm to (101.6, 129.5)
- moved 1K1 15.5 mm to (132.1, 91.4), turned to 90 degrees
- moved D3 10.5 mm to (127.0, 91.4)
- moved R10 10.2 mm to (143.9, 91.4)
- moved R11 10.2 mm to (138.8, 91.4)
- moved Q2 8.44 mm to (86.6, 127.0)
- moved R16 8.03 mm to (104.1, 134.6)
- moved Q9 7.62 mm to (106.7, 129.5)
- moved R1 5.91 mm to (87.3, 121.9)
- moved C4 5.08 mm to (108.4, 144.8)
- moved Q3 5.08 mm to (114.1, 134.6)
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Routing:
- net +5V: track 0.00 -> 147.9 mm, vias 0 -> 3
- net +3.3V: track 0.00 -> 128.1 mm
- net +12V: track 0.00 -> 128.0 mm
- net SENSORLED_1: track 0.00 -> 79.6 mm, vias 0 -> 6
- net MD_RESET: track 0.00 -> 78.0 mm, vias 0 -> 4
- net SLEEP: track 0.00 -> 70.4 mm, vias 0 -> 2
- net MOTOR_CLOCK_R: track 0.00 -> 67.9 mm, vias 0 -> 2
- net MOTOR_CW/CCW_L: track 0.00 -> 63.0 mm
- net MOTOR_CW/CCW_R: track 0.00 -> 60.7 mm, vias 0 -> 1
- net OUTA/_L: track 0.00 -> 54.5 mm, vias 0 -> 1
- net BATTERY: track 0.00 -> 46.4 mm, vias 0 -> 2
- net I2C1_SCL: track 0.00 -> 44.3 mm, vias 0 -> 1
- net photosensor_1: track 0.00 -> 40.8 mm, vias 0 -> 2
- net OUTA_L: track 0.00 -> 40.3 mm
- net I2C1_SDA: track 0.00 -> 39.3 mm
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- added copper zone on B.Cu, net GND
- added copper zone on F.Cu, net GND
