File: PCB/mouse_v1/mouse_v1.kicad_pcb (KiCad board)
At the start: 2 copper layers, 90 x 100 mm, 61 parts, among them IC1 NJM7805FA, IC2 SIT2001BI-S2-33E-12.000000G, J1 Conn_01x06_Socket, J2 Conn_01x06_Socket, J3 Conn_01x02_Socket, Q1 2SC1815GRTE2FT, Q2 2SJ681_Q_, Q3 2SJ681_Q_, Q4 ST-1KL3A, Q5 ST-1KL3A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

Commit message: 配線完了,元のデータはsensorLEDのフラグの値が両方1になっていた
Parts:
- C1, C10, C3, C6, C9: value C -> 0.1μ
- C11, C12, C2, C4, C7, C8: value C_Polarized_Small -> 100μ
- C5: value C -> 15p
- D2: value D -> BA157
- J1, J2, J3: moved to B.Cu
- R1, R10, R13, R16, R2, R3, R4: value R -> 10K
- R11, R12, R15, R5, R6, R7, R8: value R -> 4.7K
- R14, R9: value R -> 50K
- R18: value R -> 100K
- R19: value R -> 22K
- moved SW4 211.4 mm to (62.3, 76.2)
- moved Q2 209.3 mm to (66.3, 55.9)
- moved D1 205.5 mm to (67.8, 71.1)
- moved LS1 183.3 mm to (86.4, 73.7), turned to -90 degrees
- moved U2 183.3 mm to (78.5, 118.1), turned to 90 degrees
- moved R18 181.4 mm to (68.6, 61.0)
- moved C3 180.2 mm to (62.7, 66.0)
- moved C4 179.7 mm to (62.7, 71.1)
- moved J3 177.8 mm to (76.2, 86.4), turned to -90 degrees
- moved VR1 174.9 mm to (91.4, 129.5), turned to -90 degrees
- moved Q9 174.1 mm to (101.6, 78.7)
- moved R19 172.7 mm to (77.8, 61.0)
- moved D2 172.4 mm to (100.8, 71.1)
- moved R1 172.1 mm to (67.7, 66.0)
- moved Q3 171.6 mm to (101.8, 129.5)
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- renumbered R17 to 1K1
Connections:
- R11 pad 2: SENSORLED_1 -> SENSORLED_2
Routing:
- net +5V: track 0.00 -> 242.2 mm, vias 0 -> 9
- net +12V: track 0.00 -> 230.9 mm, vias 0 -> 5
- net +3.3V: track 0.00 -> 223.6 mm, vias 0 -> 8
- net photosensor_1: track 0.00 -> 95.6 mm, vias 0 -> 3
- net MD_RESET: track 0.00 -> 74.6 mm, vias 0 -> 2
- net SLEEP: track 0.00 -> 71.1 mm, vias 0 -> 2
- net BATTERY: track 0.00 -> 69.8 mm, vias 0 -> 2
- net MOTOR_CLOCK_R: track 0.00 -> 68.1 mm
- net photosensor_2: track 0.00 -> 65.5 mm, vias 0 -> 1
- net INTERFACELED: track 0.00 -> 62.8 mm, vias 0 -> 3
- net MOTOR_CW/CCW_R: track 0.00 -> 58.7 mm
- net photosensor_4: track 0.00 -> 58.0 mm, vias 0 -> 1
- net MOTOR_CW/CCW_L: track 0.00 -> 57.1 mm
- net SWITCH_2: track 0.00 -> 55.0 mm, vias 0 -> 1
- net SWITCH_1: track 0.00 -> 53.3 mm, vias 0 -> 1
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- added copper zone on B.Cu, net GND
- added copper zone on F.Cu, net GND

Commit message: アートワークを部品ごとに区分けした
Parts:
- J1, J2, J3: moved to F.Cu
- moved LED1 277.9 mm to (345.3, 7.08), turned to 0 degrees
- moved C11 255.2 mm to (359.0, 33.7)
- moved Q1 254.4 mm to (355.5, 5.90)
- moved LED2 250.7 mm to (345.3, 16.0), turned to 0 degrees
- moved R9 244.8 mm to (355.5, 16.1)
- moved R11 234.8 mm to (355.5, 21.1)
- moved R10 234.3 mm to (355.5, 18.6)
- moved C8 194.4 mm to (277.6, 154.9)
- moved J2 180.1 mm to (266.8, 168.0), turned to 0 degrees
- moved Q2 177.4 mm to (224.7, 135.7)
- moved SW4 176.4 mm to (224.8, 144.8)
- moved DS1 171.6 mm to (272.6, 115.7)
- moved C9 156.8 mm to (283.7, 127.0)
- moved C10 156.7 mm to (283.7, 129.5)
- moved C3 154.7 mm to (197.1, 142.8)
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Connections:
- R11 pad 2: SENSORLED_2 -> SENSORLED_1
Routing:
- net +5V: track 242.2 -> 0.00 mm, vias 9 -> 0
- net +12V: track 230.9 -> 0.00 mm, vias 5 -> 0
- net +3.3V: track 223.6 -> 0.00 mm, vias 8 -> 0
- net photosensor_1: track 95.6 -> 0.00 mm, vias 3 -> 0
- net MD_RESET: track 74.6 -> 0.00 mm, vias 2 -> 0
- net SLEEP: track 71.1 -> 0.00 mm, vias 2 -> 0
- net BATTERY: track 69.8 -> 0.00 mm, vias 2 -> 0
- net MOTOR_CLOCK_R: track 68.1 -> 0.00 mm
- net photosensor_2: track 65.5 -> 0.00 mm, vias 1 -> 0
- net INTERFACELED: track 62.8 -> 0.00 mm, vias 3 -> 0
- net MOTOR_CW/CCW_R: track 58.7 -> 0.00 mm
- net photosensor_4: track 58.0 -> 0.00 mm, vias 1 -> 0
- net MOTOR_CW/CCW_L: track 57.1 -> 0.00 mm
- net SWITCH_2: track 55.0 -> 0.00 mm, vias 1 -> 0
- net SWITCH_1: track 53.3 -> 0.00 mm, vias 1 -> 0
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- removed copper zone on B.Cu, net GND
- removed copper zone on F.Cu, net GND
Other:
- board outline removed

Commit message: 配線完了(仮)
Parts:
- C11, C12, C2, C4, C7, C8: footprint Capacitor_SMD:C_0603_1608Metric -> Capacitor_THT:CP_Radial_D6.3mm_P2.50mm
- J1, J2, J3, LED1, LED2, LED3, LED4, Q4, Q5, Q6, Q7: moved to B.Cu
- Q1, Q8, Q9: footprint 2SC1815GRTE2FT:2SC1815GRTE2FT -> Package_TO_SOT_SMD:SOT-23
- moved R10 260.9 mm to (100.5, 73.6), turned to 180 degrees
- moved Q1 260.2 mm to (104.4, 74.1), turned to 180 degrees
- moved R11 257.6 mm to (104.3, 78.0)
- moved LED1 245.9 mm to (106.6, 66.3), turned to -60 degrees
- moved R9 234.9 mm to (132.9, 91.0)
- moved LED2 226.3 mm to (129.6, 84.3), turned to -10 degrees
- moved C11 225.0 mm to (139.3, 82.0)
- moved J1 187.8 mm to (79.3, 149.0), turned to 180 degrees
- moved C7 187.7 mm to (91.8, 125.5), turned to -90 degrees
- moved C10 186.3 mm to (101.8, 89.0), turned to 180 degrees
- moved C9 184.0 mm to (103.3, 90.5), turned to 180 degrees
- moved C8 180.5 mm to (99.3, 126.5), turned to -90 degrees
- moved DS1 177.2 mm to (97.8, 86.8)
- moved R14 176.1 mm to (83.8, 89.5), turned to 180 degrees
- moved LED3 170.7 mm to (70.1, 84.8), turned to 10 degrees
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Connections:
- R11 pad 2: SENSORLED_1 -> SENSORLED_2
Routing:
- net +5V: track 0.00 -> 186.0 mm, vias 0 -> 4
- net +3.3V: track 0.00 -> 183.3 mm, vias 0 -> 2
- net +12V: track 0.00 -> 159.9 mm, vias 0 -> 1
- net MD_RESET: track 0.00 -> 84.7 mm, vias 0 -> 3
- net MOTOR_CLOCK_L: track 0.00 -> 77.6 mm, vias 0 -> 2
- net SLEEP: track 0.00 -> 73.4 mm, vias 0 -> 1
- net photosensor_1: track 0.00 -> 53.2 mm
- net MOTOR_ENABLE: track 0.00 -> 49.7 mm, vias 0 -> 3
- net I2C1_SCL: track 0.00 -> 45.5 mm
- net photosensor_3: track 0.00 -> 42.4 mm
- net MOTOR_CLOCK_R: track 0.00 -> 41.0 mm, vias 0 -> 1
- net OUTA_R: track 0.00 -> 40.2 mm, vias 0 -> 1
- net photosensor_2: track 0.00 -> 40.1 mm, vias 0 -> 1
- net SPEAKER: track 0.00 -> 37.3 mm, vias 0 -> 2
- net OUTB_L: track 0.00 -> 37.2 mm, vias 0 -> 1
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- added copper zone on B.Cu, net GND
- added copper zone on F.Cu, net GND
