File: PCB/mouse_v1/_autosave-mouse_v1.kicad_pcb (KiCad board)
At the start: 2 copper layers, 90 x 100 mm, 61 parts, among them IC1 NJM7805FA, IC2 SIT2001BI-S2-33E-12.000000G, J1 Conn_01x06_Socket, J2 Conn_01x06_Socket, J3 Conn_01x02_Socket, Q1 2SC1815GRTE2FT, Q2 2SJ681_Q_, Q3 2SJ681_Q_, Q4 ST-1KL3A, Q5 ST-1KL3A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

Commit message: 未配線部分を配線した
Routing:
- net GND: vias 104 -> 107
Changed lines of the file:
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@@
+	)
+	(via
+		(at 119.02 90.8)
+		(size 0.8)
+		(drill 0.4)
+		(layers "F.Cu" "B.Cu")
+		(free yes)
+		(net 2)
 	)
 	(via
@@
 	(via
 		(at 68.38 112.9)
+		(size 0.8)
+		(drill 0.4)
+		(layers "F.Cu" "B.Cu")
+		(free yes)
+		(net 2)
+	)
+	(via
+		(at 70.85 107.16)
 		(size 0.8)
 		(drill 0.4)
@@
 		(size 0.8)
 		(drill 0.4)
+		(layers "F.Cu" "B.Cu")
+		(free yes)
+		(net 2)
+	)
+	(via
+		(at 112.54 88.37)
+		(size 0.8)
+		(drill 0.4)
